File: LNA.sch (KiCad schematic (older format))
At the start: 7 parts, among them U2 SPF5189Z

Commit message: done till all routing ground ring and ground plane handeled, only bare copper part is left
Parts:
- U2: symbol vk_custom_kicad:SBB5089Z -> rj-2-4ghz-filter-amp-rescue:SBB5089Z-vk_custom_kicad
Changed lines of the file:
@@
 	5525 3350 5975 3350
 $Comp
-L vk_custom_kicad:SBB5089Z U2
+L rj-2-4ghz-filter-amp-rescue:SBB5089Z-vk_custom_kicad U2
 U 1 1 5D702FA1
 P 5525 3950
+AR Path="/5D702FA1" Ref="U2"  Part="1"
+AR Path="/5F10D83B/5D702FA1" Ref="U2"  Part="1"
 F 0 "U2" H 6219 3996 50  0000 L CNN
 F 1 "SPF5189Z" H 6219 3905 50  0000 L CNN
