File: rf-attenuator.sch (KiCad schematic (older format))
At the start: 6 parts, among them J3 Conn_01x03, J4 Conn_01x03, J5 Conn_01x03, J6 Conn_01x03, J7 Conn_01x02, U3 RFSA3613

Commit message: done till all routing ground ring and ground plane handeled, only bare copper part is left
Parts:
- J3, J4, J5, J6: footprint Connector_PinHeader_2.54mm:PinHeader_1x03_P2.54mm_Vertical -> Connector_PinHeader_2.54mm:PinHeader_1x03_P2.54mm_Vertical_SMD_Pin1Left
- J7: footprint Connector_PinHeader_2.54mm:PinHeader_1x02_P2.54mm_Vertical -> Connector_PinHeader_2.54mm:PinHeader_1x02_P2.54mm_Vertical_SMD_Pin1Left
Changed lines of the file:
@@
 F 0 "J3" H 1543 1100 50  0000 C CNN
 F 1 "Conn_01x03" H 1543 1191 50  0000 C CNN
-F 2 "Connector_PinHeader_2.54mm:PinHeader_1x03_P2.54mm_Vertical" H 1625 1425 50  0001 C CNN
+F 2 "Connector_PinHeader_2.54mm:PinHeader_1x03_P2.54mm_Vertical_SMD_Pin1Left" H 1625 1425 50  0001 C CNN
 F 3 "~" H 1625 1425 50  0001 C CNN
 	1    1625 1425
@@
 F 0 "J4" H 2468 1100 50  0000 C CNN
 F 1 "Conn_01x03" H 2468 1191 50  0000 C CNN
-F 2 "Connector_PinHeader_2.54mm:PinHeader_1x03_P2.54mm_Vertical" H 2550 1425 50  0001 C CNN
+F 2 "Connector_PinHeader_2.54mm:PinHeader_1x03_P2.54mm_Vertical_SMD_Pin1Left" H 2550 1425 50  0001 C CNN
 F 3 "~" H 2550 1425 50  0001 C CNN
 	1    2550 1425
@@
 F 0 "J5" H 3343 1100 50  0000 C CNN
 F 1 "Conn_01x03" H 3343 1191 50  0000 C CNN
-F 2 "Connector_PinHeader_2.54mm:PinHeader_1x03_P2.54mm_Vertical" H 3425 1425 50  0001 C CNN
+F 2 "Connector_PinHeader_2.54mm:PinHeader_1x03_P2.54mm_Vertical_SMD_Pin1Left" H 3425 1425 50  0001 C CNN
 F 3 "~" H 3425 1425 50  0001 C CNN
 	1    3425 1425
@@
 F 0 "J6" H 4168 1100 50  0000 C CNN
 F 1 "Conn_01x03" H 4168 1191 50  0000 C CNN
-F 2 "Connector_PinHeader_2.54mm:PinHeader_1x03_P2.54mm_Vertical" H 4250 1425 50  0001 C CNN
+F 2 "Connector_PinHeader_2.54mm:PinHeader_1x03_P2.54mm_Vertical_SMD_Pin1Left" H 4250 1425 50  0001 C CNN
 F 3 "~" H 4250 1425 50  0001 C CNN
 	1    4250 1425
@@
 F 0 "J7" H 5218 1150 50  0000 C CNN
 F 1 "Conn_01x02" H 5218 1241 50  0000 C CNN
-F 2 "Connector_PinHeader_2.54mm:PinHeader_1x02_P2.54mm_Vertical" H 5300 1475 50  0001 C CNN
+F 2 "Connector_PinHeader_2.54mm:PinHeader_1x02_P2.54mm_Vertical_SMD_Pin1Left" H 5300 1475 50  0001 C CNN
 F 3 "~" H 5300 1475 50  0001 C CNN
 	1    5300 1475
