File: Buck_1_5v.sch (KiCad schematic (older format))
At the start: 15 parts, among them IC1 MP1584EN-LF-Z

Commit message: minor updates
Parts:
- D2: value SS34 -> B340A-13-F
Changed lines of the file:
@@
 AR Path="/5F37BD5E/5F379D12" Ref="D?"  Part="1"
 F 0 "D2" V 6604 3380 50  0000 L CNN
-F 1 "SS34" V 6695 3380 50  0000 L CNN
+F 1 "B340A-13-F" V 6695 3380 50  0000 L CNN
 F 2 "Diode_SMD:D_SMA_Handsoldering" H 6650 3300 50  0001 C CNN
 F 3 "~" H 6650 3300 50  0001 C CNN
