File: Buck_2_5v.sch (KiCad schematic (older format))
At the start: 15 parts, among them IC2 MP1584EN-LF-Z

Commit message: minor updates
Parts:
- D3: value SS34 -> B340A-13-F
Changed lines of the file:
@@
 AR Path="/5F37BD5E/5F3AE926" Ref="D3"  Part="1"
 F 0 "D3" V 6529 3705 50  0000 L CNN
-F 1 "SS34" V 6620 3705 50  0000 L CNN
+F 1 "B340A-13-F" V 6620 3705 50  0000 L CNN
 F 2 "Diode_SMD:D_SMA_Handsoldering" H 6575 3625 50  0001 C CNN
 F 3 "~" H 6575 3625 50  0001 C CNN
